File: sn.kicad_sch (KiCad schematic)
At the start: 47 parts, among them J1 220V, J2 Load, J3 USB_C_Receptacle_USB2.0_16P, J4 Conn_02x03, Q1 BTB16-600B, Q2 BC847B, SW1 RESET, SW2 BOOT, U1 LTV-814, U2 ESP32-S3-WROOM-1, U3 MOC3052M, U5 USBLC6-2SC6, U6 LM1117MP-3.3

Commit message: remove l1 l2 d4 d2
Parts:
- removed D2, D4: ESD3.3, Diode_SMD:D_SOD-923, symbol Diode:ESD9B3.3ST5G
- removed L1, L2: 220Ohm, PCM_SparkFun-Capacitor:C_0603_1608Metric, symbol PCM_SparkFun-Coil:Ferrite_470Ohm_0603_1.0A
Connections:
- net at C2.1 (+), C3.2, PS1.4 (+Vo): now also D3.2 (A)
- net at F1.2: now also D1.2 (A)
Other:
- moved on the sheet: D1, D3

Commit message: update readme.md
Other:
- title: (none) -> Smart Light
